Commit message: tsid mujoco

File: model/jet_description/urdf/dyros_jet_robot.urdf (robot description, URDF)
Before this commit: robot dyros_jet_robot, 29 links, 28 joints
Links:
- link L_AnklePitch_Link: geometry collision mesh filename=package://tsid_jet_mujoco/model/jet_description/meshes/left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; visual mesh filename=package://tsid_jet_mujoco/model/jet_description/meshes/left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
- link L_AnkleRoll_Link: geometry collision mesh filename=package://tsid_jet_mujoco/model/jet_description/meshes/ankl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; visual mesh filename=package://tsid_jet_mujoco/model/jet_description/meshes/ankl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
- link L_ElbowRoll_Link: geometry collision mesh filename=package://tsid_jet_mujoco/model/jet_description/meshes/L_El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; visual mesh filename=package://tsid_jet_mujoco/model/jet_description/meshes/L_El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
- link L_HandYaw_Link: geometry collision mesh filename=package://tsid_jet_mujoco/model/jet_description/meshes/L_Ha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; visual mesh filename=package://tsid_jet_mujoco/model/jet_description/meshes/L_Ha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
- link L_HipPitch_Link: geometry collision mesh filename=package://tsid_jet_mujoco/model/jet_description/meshes/hip_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; visual mesh filename=package://tsid_jet_mujoco/model/jet_description/meshes/hip_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
- link L_HipRoll_Link: geometry collision mesh filename=package://tsid_jet_mujoco/model/jet_description/meshes/hip_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; visual mesh filename=package://tsid_jet_mujoco/model/jet_description/meshes/hip_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
- link L_HipYaw_Link: geometry collision mesh filename=package://tsid_jet_mujoco/model/jet_description/meshes/hip_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; visual mesh filename=package://tsid_jet_mujoco/model/jet_description/meshes/hip_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
- link L_KneePitch_Link: geometry collision mesh filename=package://tsid_jet_mujoco/model/jet_description/meshes/left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; visual mesh filename=package://tsid_jet_mujoco/model/jet_description/meshes/left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
- link L_ShoulderPitch_Link: geometry collision mesh filename=package://tsid_jet_mujoco/model/jet_description/meshes/L_Sh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; visual mesh filename=package://tsid_jet_mujoco/model/jet_description/meshes/L_Sh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
- link L_ShoulderRoll_Link: geometry collision mesh filename=package://tsid_jet_mujoco/model/jet_description/meshes/L_Sh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; visual mesh filename=package://tsid_jet_mujoco/model/jet_description/meshes/L_Sh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
- link L_ShoulderYaw_Link: geometry collision mesh filename=package://tsid_jet_mujoco/model/jet_description/meshes/L_Sh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; visual mesh filename=package://tsid_jet_mujoco/model/jet_description/meshes/L_Sh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
- link L_WristRoll_Link: geometry collision mesh filename=package://tsid_jet_mujoco/model/jet_description/meshes/L_Wr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; visual mesh filename=package://tsid_jet_mujoco/model/jet_description/meshes/L_Wr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
- link L_WristYaw_Link: geometry collision mesh filename=package://tsid_jet_mujoco/model/jet_description/meshes/L_Wr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; visual mesh filename=package://tsid_jet_mujoco/model/jet_description/meshes/L_Wr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
- link R_AnklePitch_Link: geometry collision mesh filename=package://tsid_jet_mujoco/model/jet_description/meshes/righ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; visual mesh filename=package://tsid_jet_mujoco/model/jet_description/meshes/righ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
- link R_AnkleRoll_Link: geometry collision mesh filename=package://tsid_jet_mujoco/model/jet_description/meshes/ankl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; visual mesh filename=package://tsid_jet_mujoco/model/jet_description/meshes/ankl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
- link R_ElbowRoll_Link: geometry collision mesh filename=package://tsid_jet_mujoco/model/jet_description/meshes/R_El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; visual mesh filename=package://tsid_jet_mujoco/model/jet_description/meshes/R_El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
- link R_HandYaw_Link: geometry collision mesh filename=package://tsid_jet_mujoco/model/jet_description/meshes/R_Ha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; visual mesh filename=package://tsid_jet_mujoco/model/jet_description/meshes/R_Ha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
- link R_HipPitch_Link: geometry collision mesh filename=package://tsid_jet_mujoco/model/jet_description/meshes/hip_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; visual mesh filename=package://tsid_jet_mujoco/model/jet_description/meshes/hip_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
- link R_HipRoll_Link: geometry collision mesh filename=package://tsid_jet_mujoco/model/jet_description/meshes/hip_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; visual mesh filename=package://tsid_jet_mujoco/model/jet_description/meshes/hip_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
- link R_HipYaw_Link: geometry collision mesh filename=package://tsid_jet_mujoco/model/jet_description/meshes/hip_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; visual mesh filename=package://tsid_jet_mujoco/model/jet_description/meshes/hip_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
- link R_KneePitch_Link: geometry collision mesh filename=package://tsid_jet_mujoco/model/jet_description/meshes/righ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; visual mesh filename=package://tsid_jet_mujoco/model/jet_description/meshes/righ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
- link R_ShoulderPitch_Link: geometry collision mesh filename=package://tsid_jet_mujoco/model/jet_description/meshes/R_Sh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; visual mesh filename=package://tsid_jet_mujoco/model/jet_description/meshes/R_Sh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
- link R_ShoulderRoll_Link: geometry collision mesh filename=package://tsid_jet_mujoco/model/jet_description/meshes/R_Sh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; visual mesh filename=package://tsid_jet_mujoco/model/jet_description/meshes/R_Sh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
- link R_ShoulderYaw_Link: geometry collision mesh filename=package://tsid_jet_mujoco/model/jet_description/meshes/R_Sh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; visual mesh filename=package://tsid_jet_mujoco/model/jet_description/meshes/R_Sh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
- link R_WristRoll_Link: geometry collision mesh filename=package://tsid_jet_mujoco/model/jet_description/meshes/R_Wr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; visual mesh filename=package://tsid_jet_mujoco/model/jet_description/meshes/R_Wr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
- link R_WristYaw_Link: geometry collision mesh filename=package://tsid_jet_mujoco/model/jet_description/meshes/R_Wr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; visual mesh filename=package://tsid_jet_mujoco/model/jet_description/meshes/R_Wr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
- link WaistPitch_Link: geometry collision mesh filename=package://tsid_jet_mujoco/model/jet_description/meshes/Wais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; visual mesh filename=package://tsid_jet_mujoco/model/jet_description/meshes/Wais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
- link WaistYaw_Link: geometry collision mesh filename=package://tsid_jet_mujoco/model/jet_description/meshes/Wais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; visual mesh filename=package://tsid_jet_mujoco/model/jet_description/meshes/Wais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
- link base_link: geometry collision mesh filename=package://tsid_jet_mujoco/model/jet_description/meshes/base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; visual mesh filename=package://tsid_jet_mujoco/model/jet_description/meshes/base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
